File: hardware/OLC.brd (EAGLE design)
At the start: 65.4 x 67.6 mm, 12 parts, among them IC1 MCP23017SP, J1 61301011121

Commit message: Add 5K ohm resistor as R3
The ESP01 needs a pull-up resistor on CH_PD to boot, and previous designs were missing it.
Parts:
- added R3: 5K, resistor:0207/10
Connections:
- new net N$11: R3.1, U$1.CH_PD
- net VCC: now also R3.2
Routing:
- net N$11: track 0.00 -> 12.1 mm
- net VCC: track 80.3 -> 84.0 mm
Changed lines of the file:
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@@
 </layers>
 <board>
-<fusionsync huburn="a.cGVyc29uYWw6dWUyYTRkODY1" projecturn="a.cGVyc29uYWw6dWUyYTRkODY1I0QyMDE3MTIyOTExMDE1ODQyNg" f3durn="urn:adsk.wipprod:dm.lineage:JQVX97mdTgaV1LZUfKRKYw" pcbguid="d80df14b-4bf6-416c-b7bb-4e0e636fdeff" lastpulledtime="" lastsyncedchangeguid="" latestrevisionid="39551046-2eb7-4c4b-9486-49263edb7faa" lastsyncedrevisionid="39551046-2eb7-4c4b-9486-49263edb7faa" lastboardhashguid="9593278c-2199-9359-c70e-337f4ebc097b" lastpushedtime="2020-12-31T02:35:42Z" linktopcb3d="true"/>
+<fusionsync huburn="a.cGVyc29uYWw6dWUyYTRkODY1" projecturn="a.cGVyc29uYWw6dWUyYTRkODY1I0QyMDE3MTIyOTExMDE1ODQyNg" f3durn="urn:adsk.wipprod:dm.lineage:JQVX97mdTgaV1LZUfKRKYw" pcbguid="" lastpulledtime="" lastsyncedchangeguid="" latestrevisionid="39551046-2eb7-4c4b-9486-49263edb7faa" lastsyncedrevisionid="39551046-2eb7-4c4b-9486-49263edb7faa" lastboardhashguid="9593278c-2199-9359-c70e-337f4ebc097b" lastpushedtime="2020-12-31T02:35:42Z" linktopcb3d="true"/>
 <plain>
 <wire x1="1.905" y1="31.75" x2="67.29" y2="31.75" width="0" layer="20"/>
@@
 <attribute name="VALUE" x="8.89" y="37.465" size="0.6096" layer="27" font="vector" ratio="20"/>
 </element>
+<element name="R3" library="resistor" library_urn="urn:adsk.eagle:library:348" package="0207/10" package3d_urn="urn:adsk.eagle:package:23491/2" value="5K" x="60.198" y="68.707" smashed="yes" rot="R180">
+<attribute name="NAME" x="63.246" y="67.183" size="1.27" layer="25" ratio="10" rot="R180"/>
+<attribute name="VALUE" x="62.4586" y="69.342" size="1.27" layer="27" ratio="10" rot="R180"/>
+</element>
 </elements>
 <signals>
@@
 <wire x1="29.21" y1="67.31" x2="26.67" y2="67.31" width="0.4064" layer="16"/>
 <wire x1="48.895" y1="66.04" x2="49.53" y2="65.405" width="0.4064" layer="16"/>
-<wire x1="30.48" y1="66.04" x2="31.75" y2="66.04" width="0.4064" layer="16"/>
-<wire x1="31.75" y1="66.04" x2="48.895" y2="66.04" width="0.4064" layer="16"/>
+<wire x1="30.48" y1="66.04" x2="48.895" y2="66.04" width="0.4064" layer="16"/>
 <wire x1="29.21" y1="67.31" x2="30.48" y2="66.04" width="0.4064" layer="16"/>
 <wire x1="49.53" y1="65.405" x2="49.545" y2="65.3275" width="0.4064" layer="16"/>
@@
 <wire x1="49.53" y1="68.58" x2="49.53" y2="65.3425" width="0.4064" layer="16"/>
 <wire x1="49.53" y1="65.3425" x2="49.545" y2="65.3275" width="0.4064" layer="16"/>
+<contactref element="R3" pad="2"/>
+<wire x1="51.435" y1="68.58" x2="54.991" y2="68.58" width="0.4064" layer="1"/>
+<wire x1="54.991" y1="68.58" x2="55.118" y2="68.707" width="0.4064" layer="1"/>
 </signal>
 <signal name="PIR1">
@@
 <via x="36.068" y="96.774" extent="1-16" drill="0.508"/>
 </signal>
+<signal name="N$11">
+<contactref element="U$1" pad="CH_PD"/>
+<contactref element="R3" pad="1"/>
+<wire x1="65.278" y1="68.707" x2="58.0045" y2="68.707" width="0.4064" layer="16"/>
+<wire x1="58.0045" y1="68.707" x2="54.625" y2="65.3275" width="0.4064" layer="16"/>
+</signal>
 </signals>
